Commit message: adding camera mount and placement

File: franka_description/robots/common/camera.urdf.xacro (robot description, xacro)
@@ -1,4 +1,4 @@
 <?xml version="1.0"?>
-<robot xmlns:xacro="http://www.ros.org/wiki/xacro" name="panda_camera">
+<robot xmlns:xacro="http://www.ros.org/wiki/xacro" name="camera">
   <xacro:arg name="arm_id" default="panda"/>
   <xacro:arg name="load_gripper" default="true"/>

File: franka_description/robots/common/camera_realsense_D455.xacro (robot description, xacro)
@@ -8,5 +8,27 @@
         <origin xyz="${xyz}" rpy="${rpy}"/>
       </joint>
+      <joint name="${ns}_camera_mount" type="fixed">
+        <parent link="${connected_to}"/>
+        <child link="camera_mount"/>
+      </joint>
     </xacro:unless>
+    <link name="camera_mount">
+      <visual>
+        <geometry>
+          <mesh filename="package://franka_description/meshes/visual/camera_mount_custom_2.stl" scale="0.001 0.001 0.001"/>
+        </geometry>
+        <origin xyz="0.033 -0.066 0.107" rpy="0 0 1.57"/>
+      </visual>
+      <collision>
+        <geometry>
+          <box />
+        </geometry>
+        <origin xyz="0 0 0" rpy="0 0 0"/>
+      </collision>
+      <inertial>
+        <mass value="1" />
+        <inertia ixx="1.0" ixy="0.0" ixz="0.0" iyy="1.0" iyz="0.0" izz="1.0" />
+      </inertial>
+    </link>
     <link name="camera_realsense_D455">
       <visual>
@@ -16,10 +38,4 @@
         <origin xyz="-0.0135 0 0" rpy="0 0 0"/>
       </visual>
-      <collision>
-        <origin xyz="-0.0135 0 0" rpy="0 0 0"/>
-        <geometry>
-          <mesh filename="package://franka_description/meshes/visual/camera_realsense_D455.dae" scale="0.02 0.02 0.02"/>
-        </geometry>
-      </collision>
       <inertial>
         <mass value="1" />
