Commit message: camera extrinsic calibration

File: franka_description/robots/common/camera_realsense_D455.xacro (robot description, xacro)
@@ -14,6 +14,8 @@
           <mesh filename="package://franka_description/meshes/collision/camera_realsense_D455.stl" scale="0.02 0.02 0.02"/>
         </geometry>
+        <origin xyz="-0.0135 0 0" rpy="0 0 0"/>
       </visual>
       <collision>
+        <origin xyz="-0.0135 0 0" rpy="0 0 0"/>
         <geometry>
           <mesh filename="package://franka_description/meshes/visual/camera_realsense_D455.dae" scale="0.02 0.02 0.02"/>

File: franka_description/robots/panda/panda_camera.urdf.xacro (robot description, xacro)
@@ -10,5 +10,5 @@
   <xacro:if value="$(arg load_camera)">
     <xacro:include filename="$(find franka_description)/robots/common/camera_realsense_D455.xacro"/>
-    <xacro:camera_realsense_D455 ns="panda" xyz="0.05 -0.03 0.03" rpy="0.20 0 -2.36" connected_to="panda_link8"/>
+    <xacro:camera_realsense_D455 ns="panda" xyz="0.00 -0.078 0.1725" rpy="0 0 3.14" connected_to="panda_link7_sc"/>
   </xacro:if>
 </robot>

Commit message: collision for camera mount

File: franka_description/robots/common/camera_realsense_D455.xacro (robot description, xacro)
@@ -22,7 +22,7 @@
       <collision>
         <geometry>
-          <box />
+          <box size="0.1 0.07 0.08"/>
         </geometry>
-        <origin xyz="0 0 0" rpy="0 0 0"/>
+        <origin xyz="0 -0.06 0.13" rpy="0 0 0"/>
       </collision>
       <inertial>

Commit message: fixing collision overlap error

File: franka_description/robots/common/camera_realsense_D455.xacro (robot description, xacro)
@@ -22,7 +22,7 @@
       <collision>
         <geometry>
-          <box size="0.1 0.07 0.08"/>
+          <box size="0.1 0.06 0.062"/>
         </geometry>
-        <origin xyz="0 -0.06 0.13" rpy="0 0 0"/>
+        <origin xyz="0 -0.06 0.143" rpy="-0.1 0 0"/>
       </collision>
       <inertial>

Commit message: camera_extrinsics update using moveit_calibration & delete link_9

File: franka_description/robots/common/camera_realsense_D455.xacro (robot description, xacro)
@@ -36,5 +36,5 @@
           <mesh filename="package://franka_description/meshes/collision/camera_realsense_D455.stl" scale="0.02 0.02 0.02"/>
         </geometry>
-        <origin xyz="-0.0135 0 0" rpy="0 0 0"/>
+        <origin xyz="0 0 0" rpy="0 0 3.14"/>
       </visual>
       <inertial>
@@ -48,9 +48,10 @@
       <child link="camera_realsense_D455_gazebo_link"/>
     </joint>
-    <link name="camera_optical_link"/>
+    <!-- keep camera frame as camera_color_optical_frame so the ros plugin of the camera recognize the frame and related topics are published properly -->
+    <link name="camera_color_optical_frame"/>
     <joint name="camera_optical_joint" type="fixed">
       <origin xyz="0 0 0" rpy="0 0 0"/>
       <parent link="camera_realsense_D455_gazebo_link"/>
-      <child link="camera_optical_link"/>
+      <child link="camera_color_optical_frame"/>
     </joint>
   </xacro:macro>

File: franka_description/robots/common/franka_arm.xacro (robot description, xacro)
@@ -117,10 +117,4 @@
       <child link="${arm_id}_link8"/>
     </joint>
-    <link name="${arm_id}_link9"/>
-    <joint name="${arm_id}_link9_joint" type="fixed">
-      <origin xyz="0 0 0.103" rpy="0 0 0" />
-      <parent link="${arm_id}_link8" />
-      <child link="${arm_id}_link9" />
-    </joint>
   </xacro:macro>
 </robot>

File: franka_description/robots/common/robot_with_camera.urdf.xacro (robot description, xacro)
@@ -9,5 +9,6 @@
   <xacro:if value="$(arg load_camera)">
     <xacro:include filename="$(find franka_description)/robots/common/camera_realsense_D455.xacro"/>
-    <xacro:camera_realsense_D455 ns="$(arg arm_id)" xyz="0.00 -0.078 0.1725" rpy="0 0 3.14" connected_to="$(arg arm_id)_link7_sc"/>
+    <!-- based on moveit_calibration -->
+    <xacro:camera_realsense_D455 ns="$(arg arm_id)" xyz="0.0144624 -0.0781259 0.159075" rpy="-0.007257889863961943 -0.008755789136793268 -0.00765949205688231" connected_to="$(arg arm_id)_link7_sc"/>
   </xacro:if>
 </robot>

Commit message: camera collision fixed

File: franka_description/robots/common/camera_realsense_D455.xacro (robot description, xacro)
@@ -38,4 +38,9 @@
         <origin xyz="-0.0135 0 0" rpy="0 0 0"/>
       </visual>
+      <collision>
+        <geometry>
+          <box size="0.0 0.0 0.0"/>
+        </geometry>
+      </collision>
       <inertial>
         <mass value="1" />

Commit message: pt cloud calibration --lgtm

File: franka_description/robots/common/camera_realsense_D455.xacro (robot description, xacro)
@@ -48,10 +48,9 @@
       <child link="camera_realsense_D455_gazebo_link"/>
     </joint>
-    <!-- keep camera frame as camera_color_optical_frame so the ros plugin of the camera recognize the frame and related topics are published properly -->
-    <link name="camera_color_optical_frame"/>
-    <joint name="camera_optical_joint" type="fixed">
+    <link name="camera_color_optical_frame_0"/>
+    <joint name="camera_color_optical_joint" type="fixed">
       <origin xyz="0 0 0" rpy="0 0 0"/>
       <parent link="camera_realsense_D455_gazebo_link"/>
-      <child link="camera_color_optical_frame"/>
+      <child link="camera_color_optical_frame_0"/>
     </joint>
   </xacro:macro>

File: franka_description/robots/common/robot_with_camera.urdf.xacro (robot description, xacro)
@@ -9,6 +9,8 @@
   <xacro:if value="$(arg load_camera)">
     <xacro:include filename="$(find franka_description)/robots/common/camera_realsense_D455.xacro"/>
-    <!-- based on moveit_calibration -->
-    <xacro:camera_realsense_D455 ns="$(arg arm_id)" xyz="0.0144624 -0.0781259 0.159075" rpy="-0.007257889863961943 -0.008755789136793268 -0.00765949205688231" connected_to="$(arg arm_id)_link7_sc"/>
+    <!-- based on moveit_calibration - old calibration -->
+    <!-- <xacro:camera_realsense_D455 ns="$(arg arm_id)" xyz="0.0144624 -0.0781259 0.159075" rpy="0 0 0" connected_to="$(arg arm_id)_link7_sc"/> -->
+    <!-- point cloud calibration - tf after moveit calib of camera_link -->
+    <xacro:camera_realsense_D455 ns="$(arg arm_id)" xyz="0.002 -0.075 0.172" rpy="-0.021 -0.020 -0.026" connected_to="$(arg arm_id)_link7_sc"/>
   </xacro:if>
 </robot>

Commit message: adapt to fingertips

File: franka_description/robots/common/camera_realsense_D455.xacro (robot description, xacro)
@@ -48,9 +48,9 @@
       <child link="camera_realsense_D455_gazebo_link"/>
     </joint>
-    <link name="camera_color_optical_frame_0"/>
+    <link name="camera_color_optical_frame"/>
     <joint name="camera_color_optical_joint" type="fixed">
       <origin xyz="0 0 0" rpy="0 0 0"/>
       <parent link="camera_realsense_D455_gazebo_link"/>
-      <child link="camera_color_optical_frame_0"/>
+      <child link="camera_color_optical_frame"/>
     </joint>
   </xacro:macro>

File: franka_description/robots/common/franka_hand.xacro (robot description, xacro)
@@ -29,21 +29,4 @@
         </geometry>
       </visual>
-      <!-- end left-fingertip -->
-      <visual>
-        <origin xyz="0 0.0015 0.06" rpy="0 0 0" />
-        <geometry>
-          <box size="0.018 0.003 0.015"/>
-        </geometry>
-        <material name="Grey">
-          <color rgba="0.262 0.262 0.262 1"/>
-        </material>
-      </visual>
-      <!-- end left-fingertip collision -->
-      <collision>
-        <origin xyz="0 0.0015 0.06" rpy="0 0 0" />
-        <geometry>
-          <box size="0.018 0.003 0.015" />
-        </geometry>
-      </collision>
       <!-- screw mount -->
       <collision>
@@ -85,21 +68,4 @@
         </geometry>
       </visual>
-      <!-- end right-fingertip -->
-      <visual>
-        <origin xyz="0 -0.0015 0.06" rpy="0 0 0" />
-        <geometry>
-          <box size="0.018 0.003 0.015"/>
-        </geometry>
-        <material name="Grey">
-          <color rgba="0.262 0.262 0.262 1"/>
-        </material>
-      </visual>
-      <!-- end left-fingertip collision -->
-      <collision>
-        <origin xyz="0 -0.0015 0.06" rpy="0 0 0" />
-        <geometry>
-          <box size="0.018 0.003 0.015" />
-        </geometry>
-      </collision>
       <!-- screw mount -->
       <collision>
